Commit message: masses added

File: urdf/irobot.xacro (robot description, xacro)
@@ -27,4 +27,7 @@
                 <xacro:expandable_geometry/>
             </collision>
+            <intertial>
+                <mass value="0.2"/>
+            </intertial>
         </link>
     </xacro:macro>
@@ -44,4 +47,7 @@
                 <xacro:pipe_geometry/>
             </collision>
+             <intertial>
+                <mass value="${0.1*length}"/>
+            </intertial>
         </link>
     </xacro:macro>
@@ -60,4 +66,7 @@
                 <xacro:wheel_geometry/>
             </collision>
+             <intertial>
+                <mass value="0.2"/>
+            </intertial>
         </link>
     </xacro:macro>
@@ -77,4 +86,7 @@
             <xacro:base_link_geometry/>
         </collision>
+         <intertial>
+            <mass value="15"/>
+        </intertial>
     </link>
     <!-- expandable for upper body    -->
@@ -99,4 +111,7 @@
             <xacro:upper_body_geometry/>
         </collision>
+         <intertial>
+            <mass value="4"/>
+        </intertial>
     </link>
     <joint name="expandable_from_base_link_to_upper_body_to_upper_body" type="fixed">
@@ -136,4 +151,7 @@
                 <xacro:foot_heel_geometry/>
             </collision>
+             <intertial>
+                <mass value="0.5"/>
+            </intertial>
         </link>
         <joint name="${position}_leg_ankle_to_${position}_foot_heel" type="fixed">
@@ -163,4 +181,7 @@
                 <xacro:foot_ball_geometry/>
             </collision>
+             <intertial>
+                <mass value="0.5"/>
+            </intertial>
         </link>
         <joint name="${position}_foot_extendable_to_${position}_foot_ball" type="fixed">
@@ -250,4 +271,7 @@
             <xacro:camera_box_geometry/>
         </collision>
+         <intertial>
+            <mass value="1"/>
+        </intertial>
     </link>
     <joint name="upper_body_link_to_camera_box" type="fixed">
