Commit message: foot extendable

File: urdf/irobot.urdf (robot description, URDF)
Before this commit: robot firefighter, 9 links, 8 joints
Links:
- added link left_foot_extendable; collision cylinder length=0.2 radius=0.02; visual cylinder length=0.2 radius=0.02
- added link right_foot_extendable; collision cylinder length=0.2 radius=0.02; visual cylinder length=0.2 radius=0.02
Joints:
- removed joint left_len_ankle_to_left_foot_heel
- removed joint right_len_ankle_to_right_foot_heel
- added joint left_foot_heel_to_left_foot_extendable: type fixed, parent left_foot_heel, child left_foot_extendable, origin xyz=0 -0.25 0 rpy=1.5708 0 0
- added joint left_leg_ankle_to_left_foot_heel: type fixed, parent left_leg_ankle, child left_foot_heel, origin xyz=0 0.1 -0.2
- added joint right_foot_heel_to_right_foot_extendable: type fixed, parent right_foot_heel, child right_foot_extendable, origin xyz=0 -0.25 0 rpy=1.5708 0 0
- added joint right_leg_ankle_to_right_foot_heel: type fixed, parent right_leg_ankle, child right_foot_heel, origin xyz=0 0.1 -0.2

File: urdf/irobot.xacro (robot description, xacro)
@@ -103,8 +103,14 @@
             </collision>
         </link>
-        <joint name="${position}_len_ankle_to_${position}_foot_heel" type="fixed">
+        <joint name="${position}_leg_ankle_to_${position}_foot_heel" type="fixed">
             <parent link="${position}_leg_ankle"/>
             <child link="${position}_foot_heel"/>
             <origin xyz="0 0.1 -0.2"/>
+        </joint>
+        <xacro:expandable name="${position}_foot_extendable"/>
+        <joint name="${position}_foot_heel_to_${position}_foot_extendable" type="fixed">
+            <parent link="${position}_foot_heel"/>
+            <child link="${position}_foot_extendable"/>
+            <origin xyz="0 -0.25 0" rpy="1.5708 0 0"/>
         </joint>
     </xacro:macro>

Commit message: foot ball

File: urdf/irobot.urdf (robot description, URDF)
Before this commit: robot firefighter, 11 links, 10 joints
Links:
- added link left_foot_ball; collision box size=0.1 0.2 0.1; visual box size=0.1 0.2 0.1
- added link right_foot_ball; collision box size=0.1 0.2 0.1; visual box size=0.1 0.2 0.1
Joints:
- added joint left_foot_extendable_to_left_foot_ball: type fixed, parent left_foot_extendable, child left_foot_ball, origin xyz=0 0 0.2 rpy=1.5708 0 0
- added joint right_foot_extendable_to_right_foot_ball: type fixed, parent right_foot_extendable, child right_foot_ball, origin xyz=0 0 0.2 rpy=1.5708 0 0

File: urdf/irobot.xacro (robot description, xacro)
@@ -114,4 +114,24 @@
             <origin xyz="0 -0.25 0" rpy="1.5708 0 0"/>
         </joint>
+        <!-- foot ball-->
+        <link name="${position}_foot_ball">
+            <xacro:macro name="foot_ball_geometry">
+                <geometry>
+                    <box size="0.1 0.2 0.1"></box>
+                </geometry>
+            </xacro:macro>
+            <visual>
+                <xacro:foot_ball_geometry/>
+            </visual>
+            <collision>
+                <xacro:foot_ball_geometry/>
+            </collision>
+        </link>
+        <joint name="${position}_foot_extendable_to_${position}_foot_ball" type="fixed">
+            <parent link="${position}_foot_extendable"/>
+            <child link="${position}_foot_ball"/>
+            <!--  move rpy to the actual part instead of the joint           -->
+            <origin xyz="0 0 0.2" rpy="1.5708 0 0"/>
+        </joint>
     </xacro:macro>
     <xacro:leg position="left" parent="base_link" x_shift="0.09"/>

Commit message: rear wheel

File: urdf/irobot.urdf (robot description, URDF)
Before this commit: robot firefighter, 13 links, 12 joints
Links:
- added link left_rear_wheel; collision cylinder length=0.05 radius=0.05; visual cylinder length=0.05 radius=0.05
- added link right_rear_wheel; collision cylinder length=0.05 radius=0.05; visual cylinder length=0.05 radius=0.05
Joints:
- added joint left_foot_heel_to_left_rear_wheel: type fixed, parent left_foot_heel, child left_rear_wheel, origin xyz=0 0 -0.05 rpy=0 1.5708 0
- added joint right_foot_heel_to_right_rear_wheel: type fixed, parent right_foot_heel, child right_rear_wheel, origin xyz=0 0 -0.05 rpy=0 1.5708 0

File: urdf/irobot.xacro (robot description, xacro)
@@ -29,4 +29,19 @@
             <collision>
                 <xacro:pipe_geometry/>
+            </collision>
+        </link>
+    </xacro:macro>
+    <xacro:macro name="wheel" params="name">
+        <link name="${name}">
+            <xacro:macro name="wheel_geometry">
+                <geometry>
+                    <cylinder length="0.05" radius="0.05"/>
+                </geometry>
+            </xacro:macro>
+            <visual>
+                <xacro:wheel_geometry/>
+            </visual>
+            <collision>
+                <xacro:wheel_geometry/>
             </collision>
         </link>
@@ -134,4 +149,12 @@
             <origin xyz="0 0 0.2" rpy="1.5708 0 0"/>
         </joint>
+        <!-- rear wheel        -->
+        <xacro:wheel name="${position}_rear_wheel"/>
+        <joint name="${position}_foot_heel_to_${position}_rear_wheel" type="fixed">
+            <parent link="${position}_foot_heel"/>
+            <child link="${position}_rear_wheel"/>
+            <!--  move rpy to the actual part instead of the joint           -->
+            <origin xyz="0 0 -0.05" rpy="0 1.5708 0"/>
+        </joint>
     </xacro:macro>
     <xacro:leg position="left" parent="base_link" x_shift="0.09"/>

Commit message: front wheel

File: urdf/irobot.urdf (robot description, URDF)
Before this commit: robot firefighter, 15 links, 14 joints
Links:
- added link left_front_wheel; collision cylinder length=0.05 radius=0.05; visual cylinder length=0.05 radius=0.05
- added link right_front_wheel; collision cylinder length=0.05 radius=0.05; visual cylinder length=0.05 radius=0.05
Joints:
- added joint left_foot_ball_to_left_front_wheel: type fixed, parent left_foot_ball, child left_front_wheel, origin xyz=0 0 0.05 rpy=0 1.5708 0
- added joint right_foot_ball_to_right_front_wheel: type fixed, parent right_foot_ball, child right_front_wheel, origin xyz=0 0 0.05 rpy=0 1.5708 0

File: urdf/irobot.xacro (robot description, xacro)
@@ -157,4 +157,12 @@
             <origin xyz="0 0 -0.05" rpy="0 1.5708 0"/>
         </joint>
+        <!-- front wheel        -->
+        <xacro:wheel name="${position}_front_wheel"/>
+        <joint name="${position}_foot_ball_to_${position}_front_wheel" type="fixed">
+            <parent link="${position}_foot_ball"/>
+            <child link="${position}_front_wheel"/>
+            <!--  move rpy to the actual part instead of the joint           -->
+            <origin xyz="0 0 0.05" rpy="0 1.5708 0"/>
+        </joint>
     </xacro:macro>
     <xacro:leg position="left" parent="base_link" x_shift="0.09"/>

Commit message: arms

File: urdf/irobot.urdf (robot description, URDF)
Before this commit: robot firefighter, 17 links, 16 joints
Links:
- added link left_arm_shoulder; collision cylinder length=0.3 radius=0.02; visual cylinder length=0.3 radius=0.02
- added link right_arm_shoulder; collision cylinder length=0.3 radius=0.02; visual cylinder length=0.3 radius=0.02
Joints:
- added joint upper_body_link_to_left_arm_shoulder: type fixed, parent upper_body_link, child left_arm_shoulder, origin xyz=0.25 -0.1 0 rpy=1.5708 0 0.523599
- added joint upper_body_link_to_right_arm_shoulder: type fixed, parent upper_body_link, child right_arm_shoulder, origin xyz=-0.25 -0.1 0 rpy=1.5708 0 -0.523599

File: urdf/irobot.xacro (robot description, xacro)
@@ -168,3 +168,14 @@
     <xacro:leg position="left" parent="base_link" x_shift="0.09"/>
     <xacro:leg position="right" parent="base_link" x_shift="-0.09"/>
+    <!-- arms    -->
+    <xacro:macro name="arm" params="position parent x_shift spin">
+        <xacro:pipe name="${position}_arm_shoulder" length="0.3"/>
+        <joint name="${parent}_to_${position}_arm_shoulder" type="fixed">
+            <parent link="${parent}"/>
+            <child link="${position}_arm_shoulder"/>
+            <origin xyz="${x_shift} -0.1 0" rpy="1.5708 0 ${spin*0.523599}"/>
+        </joint>
+    </xacro:macro>
+    <xacro:arm position="left" parent="upper_body_link" x_shift="0.25" spin="1"/>
+    <xacro:arm position="right" parent="upper_body_link" x_shift="-0.25" spin="-1"/>
 </robot>

Commit message: wrists

File: urdf/irobot.urdf (robot description, URDF)
Before this commit: robot firefighter, 19 links, 18 joints
Links:
- added link left_arm_wrist; collision cylinder length=0.3 radius=0.02; visual cylinder length=0.3 radius=0.02
- added link right_arm_wrist; collision cylinder length=0.3 radius=0.02; visual cylinder length=0.3 radius=0.02
Joints:
- added joint left_arm_shoulder_to_left_arm_wrist: type fixed, parent left_arm_shoulder, child left_arm_wrist, origin xyz=0 0 0.31
- added joint right_arm_shoulder_to_right_arm_wrist: type fixed, parent right_arm_shoulder, child right_arm_wrist, origin xyz=0 0 0.31

File: urdf/irobot.xacro (robot description, xacro)
@@ -170,4 +170,5 @@
     <!-- arms    -->
     <xacro:macro name="arm" params="position parent x_shift spin">
+        <!-- shoulder        -->
         <xacro:pipe name="${position}_arm_shoulder" length="0.3"/>
         <joint name="${parent}_to_${position}_arm_shoulder" type="fixed">
@@ -176,4 +177,11 @@
             <origin xyz="${x_shift} -0.1 0" rpy="1.5708 0 ${spin*0.523599}"/>
         </joint>
+        <!-- writs        -->
+        <xacro:pipe name="${position}_arm_wrist" length="0.3"/>
+        <joint name="${position}_arm_shoulder_to_${position}_arm_wrist" type="fixed">
+            <parent link="${position}_arm_shoulder"/>
+            <child link="${position}_arm_wrist"/>
+            <origin xyz="0 0 0.31"/>
+        </joint>
     </xacro:macro>
     <xacro:arm position="left" parent="upper_body_link" x_shift="0.25" spin="1"/>

Commit message: palms and top knuckles of grippers

File: urdf/irobot.urdf (robot description, URDF)
Before this commit: robot firefighter, 21 links, 20 joints
Links:
- added link left_arm_left_gripper_top_knuckle; collision cylinder length=0.05 radius=0.005; visual cylinder length=0.05 radius=0.005
- added link left_arm_palm; collision cylinder length=0.05 radius=0.02; visual cylinder length=0.05 radius=0.02
- added link right_arm_left_gripper_top_knuckle; collision cylinder length=0.05 radius=0.005; visual cylinder length=0.05 radius=0.005
- added link right_arm_palm; collision cylinder length=0.05 radius=0.02; visual cylinder length=0.05 radius=0.02
Joints:
- added joint left_arm_palm_left_arm_left_gripper_top_knuckle: type fixed, parent left_arm_palm, child left_arm_left_gripper_top_knuckle, origin xyz=0.03 0 0.05 rpy=0 0.523599 0
- added joint left_arm_wrist_to_left_arm_palm: type fixed, parent left_arm_wrist, child left_arm_palm, origin xyz=0 0 0.19
- added joint right_arm_palm_right_arm_left_gripper_top_knuckle: type fixed, parent right_arm_palm, child right_arm_left_gripper_top_knuckle, origin xyz=0.03 0 0.05 rpy=0 0.523599 0
- added joint right_arm_wrist_to_right_arm_palm: type fixed, parent right_arm_wrist, child right_arm_palm, origin xyz=0 0 0.19

File: urdf/irobot.xacro (robot description, xacro)
@@ -17,9 +17,9 @@
         </link>
     </xacro:macro>
-    <xacro:macro name="pipe" params="name length">
+    <xacro:macro name="pipe" params="name length radius=0.02">
         <link name="${name}">
             <xacro:macro name="pipe_geometry">
                 <geometry>
-                    <cylinder length="${length}" radius="0.02"/>
+                    <cylinder length="${length}" radius="${radius}"/>
                 </geometry>
             </xacro:macro>
@@ -184,4 +184,22 @@
             <origin xyz="0 0 0.31"/>
         </joint>
+        <!-- palms        -->
+        <xacro:pipe name="${position}_arm_palm" length="0.05"/>
+        <joint name="${position}_arm_wrist_to_${position}_arm_palm" type="fixed">
+            <parent link="${position}_arm_wrist"/>
+            <child link="${position}_arm_palm"/>
+            <origin xyz="0 0 0.19"/>
+        </joint>
+        <!-- gripper        -->
+        <xacro:macro name="gripper" params="arm_position gripper_position parent pitch">
+            <!-- top knuckle           -->
+            <xacro:pipe name="${arm_position}_arm_${gripper_position}_gripper_top_knuckle" length="0.05" radius="0.005"/>
+           <joint name="${parent}_${arm_position}_arm_${gripper_position}_gripper_top_knuckle" type="fixed">
+                <parent link="${parent}"/>
+                <child link="${arm_position}_arm_${gripper_position}_gripper_top_knuckle"/>
+                <origin xyz="0.03 0 0.05" rpy="0 ${pitch} 0"/>
+            </joint>
+        </xacro:macro>
+        <xacro:gripper parent="${position}_arm_palm" arm_position="${position}" gripper_position="left" pitch="0.523599"/>
     </xacro:macro>
     <xacro:arm position="left" parent="upper_body_link" x_shift="0.25" spin="1"/>

Commit message: second knuckle

File: urdf/irobot.urdf (robot description, URDF)
Before this commit: robot firefighter, 25 links, 24 joints
Links:
- added link left_arm_left_gripper_middle_knuckle; collision cylinder length=0.05 radius=0.005; visual cylinder length=0.05 radius=0.005
- added link right_arm_left_gripper_middle_knuckle; collision cylinder length=0.05 radius=0.005; visual cylinder length=0.05 radius=0.005
Joints:
- added joint left_arm_left_gripper_top_knuckle_to_left_arm_left_gripper_middle_knuckle: type fixed, parent left_arm_left_gripper_top_knuckle, child left_arm_left_gripper_middle_knuckle, origin xyz=-0.02 0 0.02 rpy=0 -1.5708 0
- added joint right_arm_left_gripper_top_knuckle_to_right_arm_left_gripper_middle_knuckle: type fixed, parent right_arm_left_gripper_top_knuckle, child right_arm_left_gripper_middle_knuckle, origin xyz=-0.02 0 0.02 rpy=0 -1.5708 0

File: urdf/irobot.xacro (robot description, xacro)
@@ -200,4 +200,11 @@
                 <origin xyz="0.03 0 0.05" rpy="0 ${pitch} 0"/>
             </joint>
+            <!-- middle knuckle           -->
+            <xacro:pipe name="${arm_position}_arm_${gripper_position}_gripper_middle_knuckle" length="0.05" radius="0.005"/>
+           <joint name="${arm_position}_arm_${gripper_position}_gripper_top_knuckle_to_${arm_position}_arm_${gripper_position}_gripper_middle_knuckle" type="fixed">
+                <parent link="${arm_position}_arm_${gripper_position}_gripper_top_knuckle"/>
+                <child link="${arm_position}_arm_${gripper_position}_gripper_middle_knuckle"/>
+                <origin xyz="-0.02 0 0.02" rpy="0 -1.5708 0"/>
+            </joint>
         </xacro:macro>
         <xacro:gripper parent="${position}_arm_palm" arm_position="${position}" gripper_position="left" pitch="0.523599"/>

Commit message: bottom knuckle

File: urdf/irobot.urdf (robot description, URDF)
Before this commit: robot firefighter, 27 links, 26 joints
Links:
- added link left_arm_left_gripper_bottom_knuckle; collision cylinder length=0.05 radius=0.005; visual cylinder length=0.05 radius=0.005
- added link right_arm_left_gripper_bottom_knuckle; collision cylinder length=0.05 radius=0.005; visual cylinder length=0.05 radius=0.005
Joints:
- added joint left_arm_left_gripper_middle_knuckle_to_left_arm_left_gripper_bottom_knuckle: type fixed, parent left_arm_left_gripper_middle_knuckle, child left_arm_left_gripper_bottom_knuckle, origin xyz=0 0 0.02 rpy=0 0.785398 0
- added joint right_arm_left_gripper_middle_knuckle_to_right_arm_left_gripper_bottom_knuckle: type fixed, parent right_arm_left_gripper_middle_knuckle, child right_arm_left_gripper_bottom_knuckle, origin xyz=0 0 0.02 rpy=0 0.785398 0

File: urdf/irobot.xacro (robot description, xacro)
@@ -207,4 +207,11 @@
                 <origin xyz="-0.02 0 0.02" rpy="0 -1.5708 0"/>
             </joint>
+            <!-- bottom knuckle           -->
+            <xacro:pipe name="${arm_position}_arm_${gripper_position}_gripper_bottom_knuckle" length="0.05" radius="0.005"/>
+           <joint name="${arm_position}_arm_${gripper_position}_gripper_middle_knuckle_to_${arm_position}_arm_${gripper_position}_gripper_bottom_knuckle" type="fixed">
+                <parent link="${arm_position}_arm_${gripper_position}_gripper_middle_knuckle"/>
+                <child link="${arm_position}_arm_${gripper_position}_gripper_bottom_knuckle"/>
+                <origin xyz="0 0 0.02" rpy="0 0.785398 0"/>
+            </joint>
         </xacro:macro>
         <xacro:gripper parent="${position}_arm_palm" arm_position="${position}" gripper_position="left" pitch="0.523599"/>
