Commit message: bug fixes

File: urdf/irobot.urdf (robot description, URDF)
Before this commit: robot firefighter, 29 links, 28 joints
Links:
- removed link left_arm_left_gripper_bottom_knuckle
- removed link right_arm_left_gripper_bottom_knuckle
- added link left_arm_bottom_gripper_middle_knuckle; collision cylinder length=0.05 radius=0.005; visual cylinder length=0.05 radius=0.005
- added link left_arm_bottom_gripper_top_knuckle; collision cylinder length=0.05 radius=0.005; visual cylinder length=0.05 radius=0.005
- added link left_arm_right_gripper_middle_knuckle; collision cylinder length=0.05 radius=0.005; visual cylinder length=0.05 radius=0.005
- added link left_arm_right_gripper_top_knuckle; collision cylinder length=0.05 radius=0.005; visual cylinder length=0.05 radius=0.005
- added link right_arm_bottom_gripper_middle_knuckle; collision cylinder length=0.05 radius=0.005; visual cylinder length=0.05 radius=0.005
- added link right_arm_bottom_gripper_top_knuckle; collision cylinder length=0.05 radius=0.005; visual cylinder length=0.05 radius=0.005
- added link right_arm_right_gripper_middle_knuckle; collision cylinder length=0.05 radius=0.005; visual cylinder length=0.05 radius=0.005
- added link right_arm_right_gripper_top_knuckle; collision cylinder length=0.05 radius=0.005; visual cylinder length=0.05 radius=0.005
Joints:
- removed joint left_arm_left_gripper_middle_knuckle_to_left_arm_left_gripper_bottom_knuckle
- removed joint right_arm_left_gripper_middle_knuckle_to_right_arm_left_gripper_bottom_knuckle
- added joint left_arm_bottom_gripper_top_knuckle_to_left_arm_bottom_gripper_middle_knuckle: type fixed, parent left_arm_bottom_gripper_top_knuckle, child left_arm_bottom_gripper_middle_knuckle, origin xyz=0 0 0.05 rpy=0 -1.047201225112 0
- added joint left_arm_palm_left_arm_bottom_gripper_top_knuckle: type fixed, parent left_arm_palm, child left_arm_bottom_gripper_top_knuckle, origin xyz=0 0 0.05 rpy=0 0.523599 -1.5708
- added joint left_arm_palm_left_arm_right_gripper_top_knuckle: type fixed, parent left_arm_palm, child left_arm_right_gripper_top_knuckle, origin xyz=0 0 0.05 rpy=0 0.523599 3.14159
- added joint left_arm_right_gripper_top_knuckle_to_left_arm_right_gripper_middle_knuckle: type fixed, parent left_arm_right_gripper_top_knuckle, child left_arm_right_gripper_middle_knuckle, origin xyz=0 0 0.05 rpy=0 -1.047201225112 0
- added joint right_arm_bottom_gripper_top_knuckle_to_right_arm_bottom_gripper_middle_knuckle: type fixed, parent right_arm_bottom_gripper_top_knuckle, child right_arm_bottom_gripper_middle_knuckle, origin xyz=0 0 0.05 rpy=0 -1.047201225112 0
- added joint right_arm_palm_right_arm_bottom_gripper_top_knuckle: type fixed, parent right_arm_palm, child right_arm_bottom_gripper_top_knuckle, origin xyz=0 0 0.05 rpy=0 0.523599 -1.5708
- added joint right_arm_palm_right_arm_right_gripper_top_knuckle: type fixed, parent right_arm_palm, child right_arm_right_gripper_top_knuckle, origin xyz=0 0 0.05 rpy=0 0.523599 3.14159
- added joint right_arm_right_gripper_top_knuckle_to_right_arm_right_gripper_middle_knuckle: type fixed, parent right_arm_right_gripper_top_knuckle, child right_arm_right_gripper_middle_knuckle, origin xyz=0 0 0.05 rpy=0 -1.047201225112 0
- joint base_link_to_expandable_to_upper_body: origin xyz=0 0 0.3  -> xyz=0 0 0.4 
- joint base_link_to_left_leg_hip: origin xyz=0.09 0 -0.35 -> xyz=0.09 0 -0.2
- joint base_link_to_right_leg_hip: origin xyz=-0.09 0 -0.35 -> xyz=-0.09 0 -0.2
- joint expandable_from_base_link_to_upper_body_to_upper_body: origin xyz=0 0 0.2 -> xyz=0 0 0.1
- joint left_arm_left_gripper_top_knuckle_to_left_arm_left_gripper_middle_knuckle: origin xyz=-0.02 0 0.02 rpy=0 -1.5708 0 -> xyz=0 0 0.05 rpy=0 -1.047201225112 0
- joint left_arm_palm_left_arm_left_gripper_top_knuckle: origin xyz=0.03 0 0.05 rpy=0 0.523599 0 -> xyz=0 0 0.05 rpy=0 0.523599 0
- joint left_arm_wrist_to_left_arm_palm: origin xyz=0 0 0.19 -> xyz=0 0 0.31
- joint left_foot_ball_to_left_front_wheel: origin xyz=0 0 0.05 rpy=0 1.5708 0 -> xyz=0 0 0.1 rpy=0 1.5708 0
- joint left_foot_extendable_to_left_foot_ball: origin xyz=0 0 0.2 rpy=1.5708 0 0 -> xyz=0 0.05 0.1 rpy=1.5708 0 0
- joint left_foot_heel_to_left_foot_extendable: origin xyz=0 -0.25 0 rpy=1.5708 0 0 -> xyz=0 -0.35 -0.05 rpy=1.5708 0 0
- joint left_foot_heel_to_left_rear_wheel: origin xyz=0 0 -0.05 rpy=0 1.5708 0 -> xyz=0 0 -0.1 rpy=0 1.5708 0
- joint left_leg_ankle_to_left_foot_heel: origin xyz=0 0.1 -0.2 -> xyz=0 0.1 -0.31
- joint right_arm_left_gripper_top_knuckle_to_right_arm_left_gripper_middle_knuckle: origin xyz=-0.02 0 0.02 rpy=0 -1.5708 0 -> xyz=0 0 0.05 rpy=0 -1.047201225112 0
- joint right_arm_palm_right_arm_left_gripper_top_knuckle: origin xyz=0.03 0 0.05 rpy=0 0.523599 0 -> xyz=0 0 0.05 rpy=0 0.523599 0
- joint right_arm_wrist_to_right_arm_palm: origin xyz=0 0 0.19 -> xyz=0 0 0.31
- joint right_foot_ball_to_right_front_wheel: origin xyz=0 0 0.05 rpy=0 1.5708 0 -> xyz=0 0 0.1 rpy=0 1.5708 0
- joint right_foot_extendable_to_right_foot_ball: origin xyz=0 0 0.2 rpy=1.5708 0 0 -> xyz=0 0.05 0.1 rpy=1.5708 0 0
- joint right_foot_heel_to_right_foot_extendable: origin xyz=0 -0.25 0 rpy=1.5708 0 0 -> xyz=0 -0.35 -0.05 rpy=1.5708 0 0
- joint right_foot_heel_to_right_rear_wheel: origin xyz=0 0 -0.05 rpy=0 1.5708 0 -> xyz=0 0 -0.1 rpy=0 1.5708 0
- joint right_leg_ankle_to_right_foot_heel: origin xyz=0 0.1 -0.2 -> xyz=0 0.1 -0.31
- joint upper_body_link_to_left_arm_shoulder: origin xyz=0.25 -0.1 0 rpy=1.5708 0 0.523599 -> xyz=0.17 0 0 rpy=1.5708 0 0.523599
- joint upper_body_link_to_right_arm_shoulder: origin xyz=-0.25 -0.1 0 rpy=1.5708 0 -0.523599 -> xyz=-0.17 0 0 rpy=1.5708 3.14159 -0.523599

File: urdf/irobot.xacro (robot description, xacro)
@@ -1,4 +1,14 @@
 <?xml version="1.0"?>
 <robot xmlns:xacro="http://www.ros.org/wiki/xacro" name="firefighter">
+    <!-- MATERIALS    -->
+    <xacro:macro name="color" params="name rgba">
+        <material name="${name}">
+            <color rgba="${rgba}" />
+        </material>
+    </xacro:macro>
+    <!-- correct colors   -->
+    <xacro:color name="aluminium" rgba="1 0 0 1"/>
+    <xacro:color name="blue" rgba="0 0 1 1"/>
+    <xacro:color name="black" rgba="1 0 0 1"/>
     <!--    COMMON DEFINITION-->
     <xacro:macro name="expandable" params="name">
@@ -8,7 +18,9 @@
                     <cylinder length="0.2" radius="0.02"/>
                 </geometry>
+                <origin xyz="0 0 ${-0.2/2}"/>
             </xacro:macro>
             <visual>
                 <xacro:expandable_geometry/>
+                <material name="aluminium"/>
             </visual>
             <collision>
@@ -17,5 +29,5 @@
         </link>
     </xacro:macro>
-    <xacro:macro name="pipe" params="name length radius=0.02">
+    <xacro:macro name="pipe" params="name length radius=0.02 spin=-1">
         <link name="${name}">
             <xacro:macro name="pipe_geometry">
@@ -23,7 +35,9 @@
                     <cylinder length="${length}" radius="${radius}"/>
                 </geometry>
+                <origin xyz="0 0 ${spin*length/2}"/>
             </xacro:macro>
             <visual>
                 <xacro:pipe_geometry/>
+                <material name="aluminium"/>
             </visual>
             <collision>
@@ -41,4 +55,5 @@
             <visual>
                 <xacro:wheel_geometry/>
+                <material name="black"/>
             </visual>
             <collision>
@@ -57,4 +72,5 @@
         <visual>
             <xacro:base_link_geometry/>
+            <material name="blue"/>
         </visual>
         <collision>
@@ -67,5 +83,5 @@
         <parent link="base_link"/>
         <child link="expandable_from_base_link_to_upper_body"/>
-        <origin xyz="0 0 0.3 "/>
+        <origin xyz="0 0 0.4 "/>
     </joint>
     <!-- upper body    -->
@@ -78,4 +94,5 @@
         <visual>
             <xacro:upper_body_geometry/>
+            <material name="blue"/>
         </visual>
         <collision>
@@ -86,8 +103,8 @@
         <parent link="expandable_from_base_link_to_upper_body"/>
         <child link="upper_body_link"/>
-        <origin xyz="0 0 0.2"/>
+        <origin xyz="0 0 0.1"/>
     </joint>
     <!-- legs    -->
-    <xacro:macro name="leg" params="position parent x_shift">
+    <xacro:macro name="leg" params="position parent x_shift z_shift">
         <!-- hip       -->
         <xacro:pipe name="${position}_leg_hip" length="0.3"/>
@@ -95,5 +112,5 @@
             <parent link="${parent}"/>
             <child link="${position}_leg_hip"/>
-            <origin xyz="${x_shift} 0 -0.35"/>
+            <origin xyz="${x_shift} 0 ${z_shift}"/>
         </joint>
         <!-- ankle        -->
@@ -110,7 +127,9 @@
                     <box size="0.1 0.3 0.1"></box>
                 </geometry>
+                <origin xyz="0 0 -0.05"/>
             </xacro:macro>
             <visual>
                 <xacro:foot_heel_geometry/>
+                <material name="blue"/>
             </visual>
             <collision>
@@ -121,5 +140,5 @@
             <parent link="${position}_leg_ankle"/>
             <child link="${position}_foot_heel"/>
-            <origin xyz="0 0.1 -0.2"/>
+            <origin xyz="0 0.1 -0.31"/>
         </joint>
         <xacro:expandable name="${position}_foot_extendable"/>
@@ -127,5 +146,5 @@
             <parent link="${position}_foot_heel"/>
             <child link="${position}_foot_extendable"/>
-            <origin xyz="0 -0.25 0" rpy="1.5708 0 0"/>
+            <origin xyz="0 -0.35 -0.05" rpy="1.5708 0 0"/>
         </joint>
         <!-- foot ball-->
@@ -135,7 +154,9 @@
                     <box size="0.1 0.2 0.1"></box>
                 </geometry>
+                <origin xyz="0 0 0.05"/>
             </xacro:macro>
             <visual>
                 <xacro:foot_ball_geometry/>
+                <material name="blue"/>
             </visual>
             <collision>
@@ -147,5 +168,5 @@
             <child link="${position}_foot_ball"/>
             <!--  move rpy to the actual part instead of the joint           -->
-            <origin xyz="0 0 0.2" rpy="1.5708 0 0"/>
+            <origin xyz="0 0.05 0.1" rpy="1.5708 0 0"/>
         </joint>
         <!-- rear wheel        -->
@@ -155,5 +176,5 @@
             <child link="${position}_rear_wheel"/>
             <!--  move rpy to the actual part instead of the joint           -->
-            <origin xyz="0 0 -0.05" rpy="0 1.5708 0"/>
+            <origin xyz="0 0 -0.1" rpy="0 1.5708 0"/>
         </joint>
         <!-- front wheel        -->
@@ -163,20 +184,20 @@
             <child link="${position}_front_wheel"/>
             <!--  move rpy to the actual part instead of the joint           -->
-            <origin xyz="0 0 0.05" rpy="0 1.5708 0"/>
-        </joint>
-    </xacro:macro>
-    <xacro:leg position="left" parent="base_link" x_shift="0.09"/>
-    <xacro:leg position="right" parent="base_link" x_shift="-0.09"/>
+            <origin xyz="0 0 0.1" rpy="0 1.5708 0"/>
+        </joint>
+    </xacro:macro>
+    <xacro:leg position="left" parent="base_link" x_shift="0.09" z_shift="-0.2"/>
+    <xacro:leg position="right" parent="base_link" x_shift="-0.09" z_shift="-0.2"/>
     <!-- arms    -->
-    <xacro:macro name="arm" params="position parent x_shift spin">
+    <xacro:macro name="arm" params="position parent x_shift spin pitch=0">
         <!-- shoulder        -->
-        <xacro:pipe name="${position}_arm_shoulder" length="0.3"/>
+        <xacro:pipe name="${position}_arm_shoulder" length="0.3" spin="1"/>
         <joint name="${parent}_to_${position}_arm_shoulder" type="fixed">
             <parent link="${parent}"/>
             <child link="${position}_arm_shoulder"/>
-            <origin xyz="${x_shift} -0.1 0" rpy="1.5708 0 ${spin*0.523599}"/>
+            <origin xyz="${x_shift} 0 0" rpy="1.5708 ${pitch} ${spin*0.523599}"/>
         </joint>
         <!-- writs        -->
-        <xacro:pipe name="${position}_arm_wrist" length="0.3"/>
+        <xacro:pipe name="${position}_arm_wrist" length="0.3" spin="1"/>
         <joint name="${position}_arm_shoulder_to_${position}_arm_wrist" type="fixed">
             <parent link="${position}_arm_shoulder"/>
@@ -185,37 +206,32 @@
         </joint>
         <!-- palms        -->
-        <xacro:pipe name="${position}_arm_palm" length="0.05"/>
+        <xacro:pipe name="${position}_arm_palm" length="0.05" spin="1"/>
         <joint name="${position}_arm_wrist_to_${position}_arm_palm" type="fixed">
             <parent link="${position}_arm_wrist"/>
             <child link="${position}_arm_palm"/>
-            <origin xyz="0 0 0.19"/>
+            <origin xyz="0 0 0.31"/>
         </joint>
         <!-- gripper        -->
-        <xacro:macro name="gripper" params="arm_position gripper_position parent pitch">
+        <xacro:macro name="gripper" params="arm_position gripper_position parent yaw=0">
             <!-- top knuckle           -->
-            <xacro:pipe name="${arm_position}_arm_${gripper_position}_gripper_top_knuckle" length="0.05" radius="0.005"/>
+            <xacro:pipe name="${arm_position}_arm_${gripper_position}_gripper_top_knuckle" length="0.05" radius="0.005" spin="1"/>
            <joint name="${parent}_${arm_position}_arm_${gripper_position}_gripper_top_knuckle" type="fixed">
                 <parent link="${parent}"/>
                 <child link="${arm_position}_arm_${gripper_position}_gripper_top_knuckle"/>
-                <origin xyz="0.03 0 0.05" rpy="0 ${pitch} 0"/>
+                <origin xyz="0 0 0.05" rpy="0 0.523599 ${yaw}"/>
             </joint>
-            <!-- middle knuckle           -->
-            <xacro:pipe name="${arm_position}_arm_${gripper_position}_gripper_middle_knuckle" length="0.05" radius="0.005"/>
+            <!-- bottom knuckle           -->
+            <xacro:pipe name="${arm_position}_arm_${gripper_position}_gripper_middle_knuckle" length="0.05" radius="0.005" spin="1"/>
            <joint name="${arm_position}_arm_${gripper_position}_gripper_top_knuckle_to_${arm_position}_arm_${gripper_position}_gripper_middle_knuckle" type="fixed">
                 <parent link="${arm_position}_arm_${gripper_position}_gripper_top_knuckle"/>
                 <child link="${arm_position}_arm_${gripper_position}_gripper_middle_knuckle"/>
-                <origin xyz="-0.02 0 0.02" rpy="0 -1.5708 0"/>
-            </joint>
-            <!-- bottom knuckle           -->
-            <xacro:pipe name="${arm_position}_arm_${gripper_position}_gripper_bottom_knuckle" length="0.05" radius="0.005"/>
-           <joint name="${arm_position}_arm_${gripper_position}_gripper_middle_knuckle_to_${arm_position}_arm_${gripper_position}_gripper_bottom_knuckle" type="fixed">
-                <parent link="${arm_position}_arm_${gripper_position}_gripper_middle_knuckle"/>
-                <child link="${arm_position}_arm_${gripper_position}_gripper_bottom_knuckle"/>
-                <origin xyz="0 0 0.02" rpy="0 0.785398 0"/>
+                <origin xyz="0 0 0.05" rpy="0 -1.047201225112 0"/>
             </joint>
         </xacro:macro>
-        <xacro:gripper parent="${position}_arm_palm" arm_position="${position}" gripper_position="left" pitch="0.523599"/>
-    </xacro:macro>
-    <xacro:arm position="left" parent="upper_body_link" x_shift="0.25" spin="1"/>
-    <xacro:arm position="right" parent="upper_body_link" x_shift="-0.25" spin="-1"/>
+        <xacro:gripper parent="${position}_arm_palm" arm_position="${position}" gripper_position="left"  />
+        <xacro:gripper parent="${position}_arm_palm" arm_position="${position}" gripper_position="right" yaw="3.14159"/>
+        <xacro:gripper parent="${position}_arm_palm" arm_position="${position}" gripper_position="bottom" yaw="-1.5708"/>
+    </xacro:macro>
+    <xacro:arm position="left" parent="upper_body_link" x_shift="0.17" spin="1"/>
+    <xacro:arm position="right" parent="upper_body_link" x_shift="-0.17" spin="-1" pitch="3.14159"/>
 </robot>

Commit message: camera box

File: urdf/irobot.urdf (robot description, URDF)
Before this commit: robot firefighter, 35 links, 34 joints
Links:
- added link camera_box; collision box size=0.1 0.1 0.1; visual box size=0.1 0.1 0.1
Joints:
- added joint upper_body_link_to_camera_box: type fixed, parent upper_body_link, child camera_box, origin xyz=0 -0.2 0.1

File: urdf/irobot.xacro (robot description, xacro)
@@ -235,3 +235,24 @@
     <xacro:arm position="left" parent="upper_body_link" x_shift="0.17" spin="1"/>
     <xacro:arm position="right" parent="upper_body_link" x_shift="-0.17" spin="-1" pitch="3.14159"/>
+    <!-- camera box   -->
+    <link name="camera_box">
+         <xacro:macro name="camera_box_geometry">
+            <geometry>
+                <box size="0.1 0.1 0.1"></box>
+            </geometry>
+             <origin xyz="0 0.05 0.05"/>
+        </xacro:macro>
+        <visual>
+            <xacro:camera_box_geometry/>
+            <material name="blue"/>
+        </visual>
+        <collision>
+            <xacro:camera_box_geometry/>
+        </collision>
+    </link>
+    <joint name="upper_body_link_to_camera_box" type="fixed">
+        <parent link="upper_body_link"/>
+        <child link="camera_box"/>
+        <origin xyz="0 -0.2 0.1"/>
+    </joint>
 </robot>

Commit message: making camera turn

File: urdf/irobot.urdf (robot description, URDF)
Before this commit: robot firefighter, 36 links, 35 joints
Joints:
- joint upper_body_link_to_camera_box: axis (none) -> 0 0 1; origin xyz=0 -0.2 0.1 -> xyz=0 -0.1 0.1; type fixed -> continuous

File: urdf/irobot.xacro (robot description, xacro)
@@ -262,5 +262,5 @@
                 <box size="0.1 0.1 0.1"></box>
             </geometry>
-             <origin xyz="0 0.05 0.05"/>
+             <origin xyz="0 -0.05 0.05"/>
         </xacro:macro>
         <visual>
@@ -275,8 +275,9 @@
         </intertial>
     </link>
-    <joint name="upper_body_link_to_camera_box" type="fixed">
+    <joint name="upper_body_link_to_camera_box" type="continuous">
+        <axis xyz="0 0 1"/>
         <parent link="upper_body_link"/>
         <child link="camera_box"/>
-        <origin xyz="0 -0.2 0.1"/>
+        <origin xyz="0 -0.1 0.1"/>
     </joint>
 </robot>

Commit message: expandable to upper body join

File: urdf/irobot.urdf (robot description, URDF)
Before this commit: robot firefighter, 36 links, 35 joints
Joints:
- joint expandable_from_base_link_to_upper_body_to_upper_body: axis (none) -> 0 0 1; limit (none) -> lower=-0.1 upper=1.2 effort=1000.0 velocity=0.5; type fixed -> prismatic

File: urdf/irobot.xacro (robot description, xacro)
@@ -115,5 +115,7 @@
         </intertial>
     </link>
-    <joint name="expandable_from_base_link_to_upper_body_to_upper_body" type="fixed">
+    <joint name="expandable_from_base_link_to_upper_body_to_upper_body" type="prismatic">
+        <axis xyz="0 0 1"/>
+         <limit effort="1000.0" lower="-0.1" upper="1.2" velocity="0.5"/>
         <parent link="expandable_from_base_link_to_upper_body"/>
         <child link="upper_body_link"/>

Commit message: foot extandable joins

File: urdf/irobot.urdf (robot description, URDF)
Before this commit: robot firefighter, 36 links, 35 joints
Joints:
- joint left_foot_extendable_to_left_foot_ball: axis (none) -> 0 1 0; limit (none) -> lower=-0.1 upper=0.5 effort=1000.0 velocity=0.5; type fixed -> prismatic
- joint right_foot_extendable_to_right_foot_ball: axis (none) -> 0 1 0; limit (none) -> lower=-0.1 upper=0.5 effort=1000.0 velocity=0.5; type fixed -> prismatic

File: urdf/irobot.xacro (robot description, xacro)
@@ -187,5 +187,7 @@
             </intertial>
         </link>
-        <joint name="${position}_foot_extendable_to_${position}_foot_ball" type="fixed">
+        <joint name="${position}_foot_extendable_to_${position}_foot_ball" type="prismatic">
+            <axis xyz="0 1 0"/>
+            <limit effort="1000.0" lower="-0.1" upper="0.5" velocity="0.5"/>
             <parent link="${position}_foot_extendable"/>
             <child link="${position}_foot_ball"/>

Commit message: leg joints

File: urdf/irobot.urdf (robot description, URDF)
Before this commit: robot firefighter, 36 links, 35 joints
Joints:
- joint base_link_to_left_leg_hip: axis (none) -> 1 0 0; limit (none) -> lower=-1.5708 upper=1.5708 effort=1000.0 velocity=0.5; type fixed -> revolute
- joint base_link_to_right_leg_hip: axis (none) -> 1 0 0; limit (none) -> lower=-1.5708 upper=1.5708 effort=1000.0 velocity=0.5; type fixed -> revolute
- joint left_leg_hip_to_left_leg_ankle: axis (none) -> 1 0 0; limit (none) -> lower=-1.5708 upper=1.5708 effort=1000.0 velocity=0.5; type fixed -> revolute
- joint right_leg_hip_to_right_leg_ankle: axis (none) -> 1 0 0; limit (none) -> lower=-1.5708 upper=1.5708 effort=1000.0 velocity=0.5; type fixed -> revolute

File: urdf/irobot.xacro (robot description, xacro)
@@ -116,5 +116,5 @@
     </link>
     <joint name="expandable_from_base_link_to_upper_body_to_upper_body" type="prismatic">
-        <axis xyz="0 0 1"/>
+         <axis xyz="0 0 1"/>
          <limit effort="1000.0" lower="-0.1" upper="1.2" velocity="0.5"/>
         <parent link="expandable_from_base_link_to_upper_body"/>
@@ -126,5 +126,7 @@
         <!-- hip       -->
         <xacro:pipe name="${position}_leg_hip" length="0.3"/>
-        <joint name="${parent}_to_${position}_leg_hip" type="fixed">
+        <joint name="${parent}_to_${position}_leg_hip" type="revolute">
+            <axis xyz="1 0 0"/>
+            <limit effort="1000.0" lower="-1.5708" upper="1.5708" velocity="0.5"/>
             <parent link="${parent}"/>
             <child link="${position}_leg_hip"/>
@@ -133,5 +135,7 @@
         <!-- ankle        -->
         <xacro:pipe name="${position}_leg_ankle" length="0.3"/>
-        <joint name="${position}_leg_hip_to_${position}_leg_ankle" type="fixed">
+        <joint name="${position}_leg_hip_to_${position}_leg_ankle" type="revolute">
+            <axis xyz="1 0 0"/>
+            <limit effort="1000.0" lower="-1.5708" upper="1.5708" velocity="0.5"/>
             <parent link="${position}_leg_hip"/>
             <child link="${position}_leg_ankle"/>
