Commit message: shoulder joints

File: urdf/irobot.urdf (robot description, URDF)
Before this commit: robot firefighter, 36 links, 35 joints
Links:
- removed link left_arm_shoulder
- removed link right_arm_shoulder
- added link left_arm_shoulder_x; collision cylinder length=0.01 radius=0.02; visual cylinder length=0.01 radius=0.02
- added link left_arm_shoulder_y; collision cylinder length=0.3 radius=0.02; visual cylinder length=0.3 radius=0.02
- added link right_arm_shoulder_x; collision cylinder length=0.01 radius=0.02; visual cylinder length=0.01 radius=0.02
- added link right_arm_shoulder_y; collision cylinder length=0.3 radius=0.02; visual cylinder length=0.3 radius=0.02
Joints:
- removed joint left_arm_shoulder_to_left_arm_wrist
- removed joint right_arm_shoulder_to_right_arm_wrist
- removed joint upper_body_link_to_left_arm_shoulder
- removed joint upper_body_link_to_right_arm_shoulder
- added joint left_arm_shoulder_x_to_left_arm_shoulder_y: type revolute, parent left_arm_shoulder_x, child left_arm_shoulder_y, origin xyz=0 0 0.02, axis 0 1 0, limit lower=-1.5708 upper=1.5708 effort=1000.0 velocity=0.5
- added joint left_arm_shoulder_y_to_left_arm_wrist: type fixed, parent left_arm_shoulder_y, child left_arm_wrist, origin xyz=0 0 0.31
- added joint right_arm_shoulder_x_to_right_arm_shoulder_y: type revolute, parent right_arm_shoulder_x, child right_arm_shoulder_y, origin xyz=0 0 0.02, axis 0 1 0, limit lower=-1.5708 upper=1.5708 effort=1000.0 velocity=0.5
- added joint right_arm_shoulder_y_to_right_arm_wrist: type fixed, parent right_arm_shoulder_y, child right_arm_wrist, origin xyz=0 0 0.31
- added joint upper_body_link_to_left_arm_shoulder_x: type revolute, parent upper_body_link, child left_arm_shoulder_x, origin xyz=0.17 0 0 rpy=1.5708 0 1.5708, axis 1 0 0, limit lower=-1.5708 upper=1.5708 effort=1000.0 velocity=0.5
- added joint upper_body_link_to_right_arm_shoulder_x: type revolute, parent upper_body_link, child right_arm_shoulder_x, origin xyz=-0.17 0 0 rpy=1.5708 3.14159 -1.5708, axis 1 0 0, limit lower=-1.5708 upper=1.5708 effort=1000.0 velocity=0.5

File: urdf/irobot.xacro (robot description, xacro)
@@ -221,14 +221,24 @@
     <xacro:macro name="arm" params="position parent x_shift spin pitch=0">
         <!-- shoulder        -->
-        <xacro:pipe name="${position}_arm_shoulder" length="0.3" spin="1"/>
-        <joint name="${parent}_to_${position}_arm_shoulder" type="fixed">
+        <xacro:pipe name="${position}_arm_shoulder_x" length="0.01" spin="1"/>
+        <joint name="${parent}_to_${position}_arm_shoulder_x" type="revolute">
+            <axis xyz="1 0 0"/>
+            <limit effort="1000.0" lower="-1.5708" upper="1.5708" velocity="0.5"/>
             <parent link="${parent}"/>
-            <child link="${position}_arm_shoulder"/>
-            <origin xyz="${x_shift} 0 0" rpy="1.5708 ${pitch} ${spin*0.523599}"/>
+            <child link="${position}_arm_shoulder_x"/>
+            <origin xyz="${x_shift} 0 0" rpy="1.5708 ${pitch} ${spin*1.5708}"/>
+        </joint>
+        <xacro:pipe name="${position}_arm_shoulder_y" length="0.3" spin="1"/>
+        <joint name="${position}_arm_shoulder_x_to_${position}_arm_shoulder_y" type="revolute">
+            <axis xyz="0 1 0"/>
+            <limit effort="1000.0" lower="-1.5708" upper="1.5708" velocity="0.5"/>
+            <parent link="${position}_arm_shoulder_x"/>
+            <child link="${position}_arm_shoulder_y"/>
+            <origin xyz="0 0 0.02"/>
         </joint>
         <!-- writs        -->
         <xacro:pipe name="${position}_arm_wrist" length="0.3" spin="1"/>
-        <joint name="${position}_arm_shoulder_to_${position}_arm_wrist" type="fixed">
-            <parent link="${position}_arm_shoulder"/>
+        <joint name="${position}_arm_shoulder_y_to_${position}_arm_wrist" type="fixed">
+            <parent link="${position}_arm_shoulder_y"/>
             <child link="${position}_arm_wrist"/>
             <origin xyz="0 0 0.31"/>

Commit message: elbow joints

File: urdf/irobot.urdf (robot description, URDF)
Before this commit: robot firefighter, 38 links, 37 joints
Links:
- removed link left_arm_wrist
- removed link right_arm_wrist
- added link left_arm_wrist_x; collision cylinder length=0.01 radius=0.02; visual cylinder length=0.01 radius=0.02
- added link left_arm_wrist_y; collision cylinder length=0.3 radius=0.02; visual cylinder length=0.3 radius=0.02
- added link right_arm_wrist_x; collision cylinder length=0.01 radius=0.02; visual cylinder length=0.01 radius=0.02
- added link right_arm_wrist_y; collision cylinder length=0.3 radius=0.02; visual cylinder length=0.3 radius=0.02
Joints:
- removed joint left_arm_shoulder_y_to_left_arm_wrist
- removed joint left_arm_wrist_to_left_arm_palm
- removed joint right_arm_shoulder_y_to_right_arm_wrist
- removed joint right_arm_wrist_to_right_arm_palm
- added joint left_arm_shoulder_y_to_left_arm_wrist_x: type revolute, parent left_arm_shoulder_y, child left_arm_wrist_x, origin xyz=0 0 0.31, axis 1 0 0, limit lower=-1.5708 upper=1.5708 effort=1000.0 velocity=0.5
- added joint left_arm_wrist_x_to_left_arm_wrist_y: type revolute, parent left_arm_wrist_x, child left_arm_wrist_y, origin xyz=0 0 0.02, axis 0 1 0, limit lower=-1.5708 upper=1.5708 effort=1000.0 velocity=0.5
- added joint left_arm_wrist_y_to_left_arm_palm: type fixed, parent left_arm_wrist_y, child left_arm_palm, origin xyz=0 0 0.31
- added joint right_arm_shoulder_y_to_right_arm_wrist_x: type revolute, parent right_arm_shoulder_y, child right_arm_wrist_x, origin xyz=0 0 0.31, axis 1 0 0, limit lower=-1.5708 upper=1.5708 effort=1000.0 velocity=0.5
- added joint right_arm_wrist_x_to_right_arm_wrist_y: type revolute, parent right_arm_wrist_x, child right_arm_wrist_y, origin xyz=0 0 0.02, axis 0 1 0, limit lower=-1.5708 upper=1.5708 effort=1000.0 velocity=0.5
- added joint right_arm_wrist_y_to_right_arm_palm: type fixed, parent right_arm_wrist_y, child right_arm_palm, origin xyz=0 0 0.31

File: urdf/irobot.xacro (robot description, xacro)
@@ -238,14 +238,24 @@
         </joint>
         <!-- writs        -->
-        <xacro:pipe name="${position}_arm_wrist" length="0.3" spin="1"/>
-        <joint name="${position}_arm_shoulder_y_to_${position}_arm_wrist" type="fixed">
+        <xacro:pipe name="${position}_arm_wrist_x" length="0.01" spin="1"/>
+        <joint name="${position}_arm_shoulder_y_to_${position}_arm_wrist_x" type="revolute">
+            <axis xyz="1 0 0"/>
+            <limit effort="1000.0" lower="-1.5708" upper="1.5708" velocity="0.5"/>
             <parent link="${position}_arm_shoulder_y"/>
-            <child link="${position}_arm_wrist"/>
+            <child link="${position}_arm_wrist_x"/>
             <origin xyz="0 0 0.31"/>
+        </joint>
+        <xacro:pipe name="${position}_arm_wrist_y" length="0.3" spin="1"/>
+        <joint name="${position}_arm_wrist_x_to_${position}_arm_wrist_y" type="revolute">
+            <axis xyz="0 1 0"/>
+            <limit effort="1000.0" lower="-1.5708" upper="1.5708" velocity="0.5"/>
+            <parent link="${position}_arm_wrist_x"/>
+            <child link="${position}_arm_wrist_y"/>
+            <origin xyz="0 0 0.02"/>
         </joint>
         <!-- palms        -->
         <xacro:pipe name="${position}_arm_palm" length="0.05" spin="1"/>
-        <joint name="${position}_arm_wrist_to_${position}_arm_palm" type="fixed">
-            <parent link="${position}_arm_wrist"/>
+        <joint name="${position}_arm_wrist_y_to_${position}_arm_palm" type="fixed">
+            <parent link="${position}_arm_wrist_y"/>
             <child link="${position}_arm_palm"/>
             <origin xyz="0 0 0.31"/>

Commit message: knuckles joints

File: urdf/irobot.urdf (robot description, URDF)
Before this commit: robot firefighter, 40 links, 39 joints
Joints:
- joint left_arm_palm_left_arm_bottom_gripper_top_knuckle: axis (none) -> 0 1 0; limit (none) -> lower=0 upper=1.5708 effort=1000.0 velocity=0.5; type fixed -> revolute
- joint left_arm_palm_left_arm_left_gripper_top_knuckle: axis (none) -> 0 1 0; limit (none) -> lower=0 upper=1.5708 effort=1000.0 velocity=0.5; type fixed -> revolute
- joint left_arm_palm_left_arm_right_gripper_top_knuckle: axis (none) -> 0 1 0; limit (none) -> lower=0 upper=1.5708 effort=1000.0 velocity=0.5; type fixed -> revolute
- joint right_arm_palm_right_arm_bottom_gripper_top_knuckle: axis (none) -> 0 1 0; limit (none) -> lower=0 upper=1.5708 effort=1000.0 velocity=0.5; type fixed -> revolute
- joint right_arm_palm_right_arm_left_gripper_top_knuckle: axis (none) -> 0 1 0; limit (none) -> lower=0 upper=1.5708 effort=1000.0 velocity=0.5; type fixed -> revolute
- joint right_arm_palm_right_arm_right_gripper_top_knuckle: axis (none) -> 0 1 0; limit (none) -> lower=0 upper=1.5708 effort=1000.0 velocity=0.5; type fixed -> revolute

File: urdf/irobot.xacro (robot description, xacro)
@@ -265,5 +265,7 @@
             <!-- top knuckle           -->
             <xacro:pipe name="${arm_position}_arm_${gripper_position}_gripper_top_knuckle" length="0.05" radius="0.005" spin="1"/>
-           <joint name="${parent}_${arm_position}_arm_${gripper_position}_gripper_top_knuckle" type="fixed">
+           <joint name="${parent}_${arm_position}_arm_${gripper_position}_gripper_top_knuckle" type="revolute">
+                <axis xyz="0 1 0"/>
+                <limit effort="1000.0" lower="0" upper="1.5708" velocity="0.5"/>
                 <parent link="${parent}"/>
                 <child link="${arm_position}_arm_${gripper_position}_gripper_top_knuckle"/>

Commit message: palm joint

File: urdf/irobot.urdf (robot description, URDF)
Before this commit: robot firefighter, 40 links, 39 joints
Joints:
- joint left_arm_wrist_y_to_left_arm_palm: axis (none) -> 0 0 1; type fixed -> continuous
- joint right_arm_wrist_y_to_right_arm_palm: axis (none) -> 0 0 1; type fixed -> continuous

File: urdf/irobot.xacro (robot description, xacro)
@@ -256,5 +256,6 @@
         <!-- palms        -->
         <xacro:pipe name="${position}_arm_palm" length="0.05" spin="1"/>
-        <joint name="${position}_arm_wrist_y_to_${position}_arm_palm" type="fixed">
+        <joint name="${position}_arm_wrist_y_to_${position}_arm_palm" type="continuous">
+            <axis xyz="0 0 1"/>
             <parent link="${position}_arm_wrist_y"/>
             <child link="${position}_arm_palm"/>

Commit message: wheels joints

File: urdf/irobot.urdf (robot description, URDF)
Before this commit: robot firefighter, 40 links, 39 joints
Joints:
- joint left_foot_ball_to_left_front_wheel: axis (none) -> 0 0 1; type fixed -> continuous
- joint left_foot_heel_to_left_rear_wheel: axis (none) -> 0 0 1; type fixed -> continuous
- joint right_foot_ball_to_right_front_wheel: axis (none) -> 0 0 1; type fixed -> continuous
- joint right_foot_heel_to_right_rear_wheel: axis (none) -> 0 0 1; type fixed -> continuous

File: urdf/irobot.xacro (robot description, xacro)
@@ -201,5 +201,6 @@
         <!-- rear wheel        -->
         <xacro:wheel name="${position}_rear_wheel"/>
-        <joint name="${position}_foot_heel_to_${position}_rear_wheel" type="fixed">
+        <joint name="${position}_foot_heel_to_${position}_rear_wheel" type="continuous">
+            <axis xyz="0 0 1"/>
             <parent link="${position}_foot_heel"/>
             <child link="${position}_rear_wheel"/>
@@ -209,5 +210,6 @@
         <!-- front wheel        -->
         <xacro:wheel name="${position}_front_wheel"/>
-        <joint name="${position}_foot_ball_to_${position}_front_wheel" type="fixed">
+        <joint name="${position}_foot_ball_to_${position}_front_wheel" type="continuous">
+            <axis xyz="0 0 1"/>
             <parent link="${position}_foot_ball"/>
             <child link="${position}_front_wheel"/>
